File: supply-ldo-adj-single.kicad_pcb (KiCad board)
At the start: 2 copper layers, 31.8 x 33 mm, 15 parts, among them P1 CONN_02X02, P2 CONN_01X03, P3 CONN_02X08, P4 CONN_02X04, P5 CONN_01X01, P6 CONN_01X01, U1 TPS7A47

Commit message: Cleanup
Parts:
- C1: value 47uF -> T495X476K035ATE300
- C2: value 10uF -> UMK316BBJ106KL-T
- C3: value 1uF -> UMK107BJ105KA-T
- C4, C5, C6, C7, C8: value 10uF -> GRM21BR6YA106KE43L
- U1: value TPS7A47 -> TPS7A4700
Changed lines of the file:
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@@
     (links 58)
     (no_connects 2)
-    (area 71.044999 20.244999 102.945001 53.415001)
+    (area 68.551667 20.244999 105.438334 53.934)
     (thickness 1.6)
     (drawings 22)
@@
     (visible_elements FFFFFF7F)
     (pcbplotparams
-      (layerselection 0x00030_80000001)
-      (usegerberextensions false)
+      (layerselection 0x010fc_80000001)
+      (usegerberextensions true)
       (excludeedgelayer true)
       (linewidth 0.100000)
@@
       (psa4output false)
       (plotreference true)
-      (plotvalue true)
+      (plotvalue false)
       (plotinvisibletext false)
       (padsonsilk false)
@@
       (outputformat 1)
       (mirror false)
-      (drillshape 1)
+      (drillshape 0)
       (scaleselection 1)
-      (outputdirectory ""))
+      (outputdirectory gerber))
   )
   (net 0 "")
@@
       (effects (font (size 1 1) (thickness 0.15)))
     )
-    (fp_text value TPS7A47 (at 0 3.525 180) (layer F.Fab) hide
+    (fp_text value TPS7A4700 (at 0 3.525 180) (layer F.Fab) hide
       (effects (font (size 1 1) (thickness 0.15)))
     )
@@
       (effects (font (size 1 1) (thickness 0.15)))
     )
-    (fp_text value 10uF (at -5.08 0 270) (layer F.Fab) hide
+    (fp_text value UMK316BBJ106KL-T (at -5.08 0 270) (layer F.Fab) hide
       (effects (font (size 1 1) (thickness 0.15)))
     )
@@
       (effects (font (size 1 1) (thickness 0.15)))
     )
-    (fp_text value 47uF (at -1.27 -3.81) (layer F.Fab) hide
+    (fp_text value T495X476K035ATE300 (at -1.27 -3.81) (layer F.Fab) hide
       (effects (font (size 1 1) (thickness 0.15)))
     )
@@
       (effects (font (size 1 1) (thickness 0.15)))
     )
-    (fp_text value 1uF (at 0 1.9 90) (layer F.Fab) hide
+    (fp_text value UMK107BJ105KA-T (at 0 1.9 90) (layer F.Fab) hide
       (effects (font (size 1 1) (thickness 0.15)))
     )
@@
       (effects (font (size 1 1) (thickness 0.15)))
     )
-    (fp_text value 10uF (at -3.81 0 270) (layer F.Fab) hide
+    (fp_text value GRM21BR6YA106KE43L (at -3.81 0 270) (layer F.Fab) hide
       (effects (font (size 1 1) (thickness 0.15)))
     )
@@
       (effects (font (size 1 1) (thickness 0.15)))
     )
-    (fp_text value 10uF (at -3.81 0 270) (layer F.Fab) hide
+    (fp_text value GRM21BR6YA106KE43L (at -3.81 0 270) (layer F.Fab) hide
       (effects (font (size 1 1) (thickness 0.15)))
     )
@@
       (effects (font (size 1 1) (thickness 0.15)))
     )
-    (fp_text value 10uF (at -3.81 0 270) (layer F.Fab) hide
+    (fp_text value GRM21BR6YA106KE43L (at -3.81 0 270) (layer F.Fab) hide
       (effects (font (size 1 1) (thickness 0.15)))
     )
@@
       (effects (font (size 1 1) (thickness 0.15)))
     )
-    (fp_text value 10uF (at -3.81 0 270) (layer F.Fab) hide
+    (fp_text value GRM21BR6YA106KE43L (at -3.81 0 270) (layer F.Fab) hide
       (effects (font (size 1 1) (thickness 0.15)))
     )
@@
       (effects (font (size 1 1) (thickness 0.15)))
     )
-    (fp_text value 10uF (at -3.81 0 270) (layer F.Fab) hide
-      (effects (font (size 1 1) (thickness 0.15)))
-    )
+    (fp_text value GRM21BR6YA106KE43L (at -3.81 0 270) (layer F.Fab) hide
+      (effects (font (size 1 1) (thickness 0.15)))
+    )
