File: supply-ldo-adj-single.sch (KiCad schematic (older format))
At the start: 13 parts, among them P1 CONN_02X02, P2 CONN_01X03, P3 CONN_02X08, P4 CONN_02X04, U1 TPS7A47

Commit message: Add input voltage limits
Parts:
- added P5, P6: CONN_01X01, Connect:1pin, symbol CONN_01X01
- C1: footprint (none) -> Capacitors_Tantalum_SMD:TantalC_SizeD_EIA-7343_Reflow; Part (none) -> T495X476K035ATE300
- C2: footprint (none) -> Capacitors_SMD:C_1206; Part (none) -> UMK316BBJ106KL-T
- C3: footprint (none) -> Capacitors_SMD:C_0603; Part (none) -> UMK107BJ105KA-T
- C4, C5, C6, C7, C8: footprint (none) -> Capacitors_SMD:C_0805; Part (none) -> GRM21BR6YA106KE43L
- U1: value TPS7A47 -> TPS7A4700
Connections:
- net GND: now also P2.1 (P1), P3.1 (P1), P3.11 (P11), P3.13 (P13), P3.15 (P15), P3.3 (P3), P3.5 (P5), P3.7 (P7), P3.9 (P9), P4.1 (P1), P4.3 (P3), P4.5 (P5), P4.7 (P7); no longer P2.3 (P3), P3.10 (P10), P3.12 (P12), P3.14 (P14), P3.16 (P16), P3.2 (P2), P3.4 (P4), P3.6 (P6), P3.8 (P8), P4.2 (P2), P4.4 (P4), P4.6 (P6), P4.8 (P8)
- net Vout: now reaches C4.1, C5.1, C6.1, C7.1, C8.1, U1.1 (OUT), U1.20 (OUT), U1.3 (SENSE/FB)
- net Vout: now also P4.2 (P2), P4.4 (P4), P4.6 (P6), P4.8 (P8); no longer P4.1 (P1), P4.3 (P3), P4.5 (P5), P4.7 (P7)
- net at U1.10 (0P4V): now also P3.6 (P6); no longer P3.5 (P5)
- net at U1.11 (0P2V): now also P3.4 (P4); no longer P3.3 (P3)
- net at U1.12 (0P1V): now also P3.2 (P2); no longer P3.1 (P1)
- net Vin: now reaches C1.1, C2.1, P1.2 (P2), P1.4 (P4), U1.15 (IN), U1.16 (IN)
- net Vin: now also P2.3 (P3); no longer P2.1 (P1)
- net at U1.4 (6P4V2): now also P3.16 (P16); no longer P3.15 (P15)
- net at U1.5 (6P4V1): now also P3.14 (P14); no longer P3.13 (P13)
- net at U1.6 (3P2V): now also P3.12 (P12); no longer P3.11 (P11)
- net at U1.8 (1P6V): now also P3.10 (P10); no longer P3.9 (P9)
- net at U1.9 (0P8V): now also P3.8 (P8); no longer P3.7 (P7)
- no-connect marks 0 -> 2
Other:
- note added: "3≤Vin≤36"
- moved on the sheet: C1, C2, C3, C4, P1, P2, P3, P4, U1

Commit message: Cleanup
Parts:
- C1: value 47uF -> T495X476K035ATE300; Part T495X476K035ATE300 -> 47uF
- C2: value 10uF -> UMK316BBJ106KL-T; Part UMK316BBJ106KL-T -> 10uF
- C3: value 1uF -> UMK107BJ105KA-T; Part UMK107BJ105KA-T -> 1uF
- C4: value 10uF -> GRM21BR6YA106KE43L; Part GRM21BR6YA106KE43L -> 10uf
- C5, C6, C7, C8: value 10uF -> GRM21BR6YA106KE43L; Part GRM21BR6YA106KE43L -> 10uF
- U1: value TPS7A4700 -> TPS7A4700RGWR
Changed lines of the file:
@@
 P 2550 1500
 F 0 "U1" H 2600 1650 60  0000 C CNN
-F 1 "TPS7A4700" H 2800 1550 60  0000 C CNN
+F 1 "TPS7A4700RGWR" H 2900 1550 60  0000 C CNN
 F 2 "Housings_DFN_QFN:QFN-20-1EP_5x5mm_Pitch0.65mm" H 2750 1550 60  0001 C CNN
 F 3 "" H 2750 1550 60  0000 C CNN
@@
 P 4350 1850
 F 0 "C4" H 4375 1950 50  0000 L CNN
-F 1 "10uF" H 4375 1750 50  0000 L CNN
+F 1 "GRM21BR6YA106KE43L" H 4375 1750 50  0001 L CNN
 F 2 "Capacitors_SMD:C_0805" H 4388 1700 50  0001 C CNN
 F 3 "" H 4350 1850 50  0000 C CNN
-F 4 "GRM21BR6YA106KE43L" H 4350 1850 60  0001 C CNN "Part"
+F 4 "10uf" H 4450 1750 50  0000 C CNN "Part"
 	1    4350 1850
 	1    0    0    -1
@@
 P 2050 2250
 F 0 "C3" H 2075 2350 50  0000 L CNN
-F 1 "1uF" H 2075 2150 50  0000 L CNN
+F 1 "UMK107BJ105KA-T" H 2075 2150 50  0001 L CNN
 F 2 "Capacitors_SMD:C_0603" H 2088 2100 50  0001 C CNN
 F 3 "" H 2050 2250 50  0000 C CNN
-F 4 "UMK107BJ105KA-T" H 2050 2250 60  0001 C CNN "Part"
+F 4 "1uF" H 2150 2150 50  0000 C CNN "Part"
 	1    2050 2250
 	1    0    0    -1
@@
 P 1800 1850
 F 0 "C2" H 1825 1950 50  0000 L CNN
-F 1 "10uF" H 1825 1750 50  0000 L CNN
+F 1 "UMK316BBJ106KL-T" H 1825 1750 50  0001 L CNN
 F 2 "Capacitors_SMD:C_1206" H 1838 1700 50  0001 C CNN
 F 3 "" H 1800 1850 50  0000 C CNN
-F 4 "UMK316BBJ106KL-T" H 1800 1850 60  0001 C CNN "Part"
+F 4 "10uF" H 1900 1750 50  0000 C CNN "Part"
 	1    1800 1850
 	1    0    0    -1
@@
 P 1550 1850
 F 0 "C1" H 1575 1950 50  0000 L CNN
-F 1 "47uF" H 1575 1750 50  0000 L CNN
+F 1 "T495X476K035ATE300" H 1575 1750 50  0001 L CNN
 F 2 "Capacitors_Tantalum_SMD:TantalC_SizeD_EIA-7343_Reflow" H 1588 1700 50  0001 C CNN
 F 3 "" H 1550 1850 50  0000 C CNN
-F 4 "T495X476K035ATE300" H 1550 1850 60  0001 C CNN "Part"
+F 4 "47uF" H 1650 1750 50  0000 C CNN "Part"
 	1    1550 1850
 	1    0    0    -1
@@
 P 4600 1850
 F 0 "C5" H 4625 1950 50  0000 L CNN
-F 1 "10uF" H 4625 1750 50  0000 L CNN
+F 1 "GRM21BR6YA106KE43L" H 4625 1750 50  0001 L CNN
 F 2 "Capacitors_SMD:C_0805" H 4638 1700 50  0001 C CNN
 F 3 "" H 4600 1850 50  0000 C CNN
-F 4 "GRM21BR6YA106KE43L" H 4600 1850 60  0001 C CNN "Part"
+F 4 "10uF" H 4700 1750 50  0000 C CNN "Part"
 	1    4600 1850
 	1    0    0    -1
@@
 P 4850 1850
 F 0 "C6" H 4875 1950 50  0000 L CNN
-F 1 "10uF" H 4875 1750 50  0000 L CNN
+F 1 "GRM21BR6YA106KE43L" H 4875 1750 50  0001 L CNN
 F 2 "Capacitors_SMD:C_0805" H 4888 1700 50  0001 C CNN
 F 3 "" H 4850 1850 50  0000 C CNN
-F 4 "GRM21BR6YA106KE43L" H 4850 1850 60  0001 C CNN "Part"
+F 4 "10uF" H 4950 1750 50  0000 C CNN "Part"
 	1    4850 1850
 	1    0    0    -1
@@
 P 5100 1850
 F 0 "C7" H 5125 1950 50  0000 L CNN
-F 1 "10uF" H 5125 1750 50  0000 L CNN
+F 1 "GRM21BR6YA106KE43L" H 5125 1750 50  0001 L CNN
 F 2 "Capacitors_SMD:C_0805" H 5138 1700 50  0001 C CNN
 F 3 "" H 5100 1850 50  0000 C CNN
-F 4 "GRM21BR6YA106KE43L" H 5100 1850 60  0001 C CNN "Part"
+F 4 "10uF" H 5200 1750 50  0000 C CNN "Part"
 	1    5100 1850
 	1    0    0    -1
@@
 P 5350 1850
 F 0 "C8" H 5375 1950 50  0000 L CNN
-F 1 "10uF" H 5375 1750 50  0000 L CNN
+F 1 "GRM21BR6YA106KE43L" H 5375 1750 50  0001 L CNN
 F 2 "Capacitors_SMD:C_0805" H 5388 1700 50  0001 C CNN
 F 3 "" H 5350 1850 50  0000 C CNN
-F 4 "GRM21BR6YA106KE43L" H 5350 1850 60  0001 C CNN "Part"
+F 4 "10uF" H 5450 1750 50  0000 C CNN "Part"
 	1    5350 1850
 	1    0    0    -1

Commit message: Clean up
Parts:
- C2: value UMK316BBJ106KL-T -> UMK316BBJ106ML-T
Changed lines of the file:
@@
 P 1800 1850
 F 0 "C2" H 1825 1950 50  0000 L CNN
-F 1 "UMK316BBJ106KL-T" H 1825 1750 50  0001 L CNN
+F 1 "UMK316BBJ106ML-T" H 1825 1750 50  0001 L CNN
 F 2 "Capacitors_SMD:C_1206" H 1838 1700 50  0001 C CNN
 F 3 "" H 1800 1850 50  0000 C CNN

Commit message: Correct Vref to 1.4v
Other:
- note added: "Vref = 1.4V\nVout = Vref + Vadj"
- note removed: "Vref = 1.6V\nVout = Vref + Vadj"
Changed lines of the file:
@@
 	2050 2000 2350 2000
 Text Notes 2550 3000 0    60   ~ 0
-Vref = 1.6V\nVout = Vref + Vadj
+Vref = 1.4V\nVout = Vref + Vadj
 Text Notes 3750 2850 0    60   ~ 0
 Vadj
